File: mag/USBtoUART.sch (KiCad schematic (older format))
At the start: 5 parts

Commit message: тестовая прошивка, замечания по плате
тестовая прошивка - обмен по usb-uart
замечания по плате - добавлены пометки для изсправления в следующих версиях
Other:
- note added: "убрать переходки из-под микросхемы (кроме земли)"
Changed lines of the file:
@@
 NoConn ~ 6300 3400
 NoConn ~ 6300 2650
+Text Notes 7000 5050 0    50   ~ 0
+убрать переходки из-под микросхемы (кроме земли)
 $EndSCHEMATC

Commit message: библиотека bmp180, замечания к схеме
Parts:
- C11, C12: symbol elements:Конденсатор_керамический -> mag-rescue:Конденсатор_керамический-elements
- DD8: symbol elements:Преобразователь_CP2102(USB-UART) -> mag-rescue:Преобразователь_CP2102(USB-UART)-elements
- R10, R11: symbol elements:Резистор_0,065Вт -> mag-rescue:Резистор_0,065Вт-elements
Changed lines of the file:
@@
 EESchema Schematic File Version 4
 LIBS:mag-cache
-EELAYER 29 0
+EELAYER 30 0
 EELAYER END
 $Descr A4 11693 8268
@@
 TX(MOSI)
 $Comp
-L elements:Преобразователь_CP2102(USB-UART) DD8
+L mag-rescue:Преобразователь_CP2102(USB-UART)-elements DD8
 U 1 1 5DC1E646
 P 4500 2500
@@
 $EndComp
 $Comp
-L elements:Резистор_0,065Вт R?
+L mag-rescue:Резистор_0,065Вт-elements R?
 U 1 1 5DC54381
 P 7200 3000
@@
 $EndComp
 $Comp
-L elements:Конденсатор_керамический C?
+L mag-rescue:Конденсатор_керамический-elements C?
 U 1 1 5DC6BAE6
 P 3250 2700
@@
 	3250 2650 3250 2500
 $Comp
-L elements:Конденсатор_керамический C?
+L mag-rescue:Конденсатор_керамический-elements C?
 U 1 1 5DC6D54C
 P 3250 3300
@@
 gnd
 $Comp
-L elements:Резистор_0,065Вт R?
+L mag-rescue:Резистор_0,065Вт-elements R?
 U 1 1 5DC794DF
 P 7200 2500

Commit message: инициирован переезд на ESP32
Other:
- note removed: "убрать переходки из-под микросхемы (кроме земли)"
Changed lines of the file:
@@
 EESchema Schematic File Version 4
-LIBS:mag-cache
 EELAYER 30 0
 EELAYER END
@@
 NoConn ~ 6300 3400
 NoConn ~ 6300 2650
-Text Notes 7000 5050 0    50   ~ 0
-убрать переходки из-под микросхемы (кроме земли)
 $EndSCHEMATC
