File: mag/power.sch (KiCad schematic (older format))
At the start: 20 parts

Commit message: на схеме не отражены внешняя i2c-eeprom
Parts:
- added K3: кнопка_FSMSM, N_X:Кнопка_FSMSM, symbol elements:кнопка
- added R13, R14: Резистор_0,065Вт, N_RLC:Конденсатор_SMD_0603, symbol elements:Резистор_0,065Вт
- added VT1: Транзистор_полевой_P-канал(IRLML2246TRPBF), N_VD_HL:Транзистор_IRLML6344TR_SOT-23, symbol elements:Транзистор_полевой_P-канал(IRLML2246TRPBF)
- renumbered DD7 to G2
Connections:
- net BATT_out: now also VT1.3; no longer FU1.2, R6.1, R7.1, VD4.2
- net Battery-: now also K3.2
- new net: K3.1, R13.2, R14.1, VT1.1
- new net Bat_in+: FU1.2, R13.1, R6.1, R7.1, VD4.2, VT1.2
- new net pwr_on_off: R14.2
Other:
- moved on the sheet: C10, C6, C7, C8, C9, FU1, FU2, G1, G2, L1, R6, R7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

Commit message: arduino test: adc test
Other:
- note added: "замена предохранителя на пред. с меньшим сопротивлением"
Changed lines of the file:
@@
 	4500 3750 5000 3750
 Connection ~ 5000 3750
+Text Notes 500  3800 0    50   ~ 0
+замена предохранителя на пред. с меньшим сопротивлением
 $EndSCHEMATC

Commit message: библиотека bmp180, замечания к схеме
Parts:
- C10, C6, C7, C8, C9: symbol elements:Конденсатор_керамический -> mag-rescue:Конденсатор_керамический-elements
- FU1, FU2: symbol elements:Предохранитель -> mag-rescue:Предохранитель-elements
- G1: symbol elements:стабилизатор_нерегулируемый_XC6206P302MR -> mag-rescue:стабилизатор_нерегулируемый_XC6206P302MR-elements
- G2: symbol elements:Микросхема_DCDC_step_UP_LM2703 -> mag-rescue:Микросхема_DCDC_step_UP_LM2703-elements
- K3: symbol elements:кнопка -> mag-rescue:кнопка-elements
- L1: symbol elements:Чип-индуктивность -> mag-rescue:Чип-индуктивность-elements
- R13, R14, R8, R9: symbol elements:Резистор_0,065Вт -> mag-rescue:Резистор_0,065Вт-elements
- R6, R7: symbol elements:Резистор_0,25Вт -> mag-rescue:Резистор_0,25Вт-elements
- VD1, VD2, VD3, VD4, VD5, VD6: symbol elements:Диод_шоттки -> mag-rescue:Диод_шоттки-elements
- VT1: symbol elements:Транзистор_полевой_P-канал(IRLML2246TRPBF) -> mag-rescue:Транзистор_полевой_P-канал(IRLML2246TRPBF)-elements
Changed lines of the file:
@@
 EESchema Schematic File Version 4
 LIBS:mag-cache
-EELAYER 29 0
+EELAYER 30 0
 EELAYER END
 $Descr A4 11693 8268
@@
 USB_pwr_gnd
 $Comp
-L elements:Предохранитель FU?
+L mag-rescue:Предохранитель-elements FU?
 U 1 1 5D9AEB0E
 P 2350 3500
@@
 USB_vcc
 $Comp
-L elements:Диод_шоттки VD5
+L mag-rescue:Диод_шоттки-elements VD5
 U 1 1 5DA75E76
 P 4000 1650
@@
 	3350 1000 4000 1000
 $Comp
-L elements:Диод_шоттки VD1
+L mag-rescue:Диод_шоттки-elements VD1
 U 1 1 5D9AF37D
 P 3350 1950
@@
 Connection ~ 3350 2250
 $Comp
-L elements:Резистор_0,25Вт R6
+L mag-rescue:Резистор_0,25Вт-elements R6
 U 1 1 5DA90F31
 P 3500 3500
@@
 $EndComp
 $Comp
-L elements:Резистор_0,25Вт R7
+L mag-rescue:Резистор_0,25Вт-elements R7
 U 1 1 5DA924F9
 P 3500 4000
@@
 $EndComp
 $Comp
-L elements:Диод_шоттки VD4
+L mag-rescue:Диод_шоттки-elements VD4
 U 1 1 5DA92C22
 P 3350 2700
@@
 gnd
 $Comp
-L elements:Предохранитель FU?
+L mag-rescue:Предохранитель-elements FU?
 U 1 1 5DAA0CE8
 P 2150 1000
@@
 	3350 3150 2950 3150
 $Comp
-L elements:Диод_шоттки VD3
+L mag-rescue:Диод_шоттки-elements VD3
 U 1 1 5DB56B32
 P 2650 1950
@@
 $EndComp
 $Comp
-L elements:Диод_шоттки VD2
+L mag-rescue:Диод_шоттки-elements VD2
 U 1 1 5DB57165
 P 2000 1950
@@
 	7800 3250 8000 3250
 $Comp
-L elements:Конденсатор_керамический C?
+L mag-rescue:Конденсатор_керамический-elements C?
 U 1 1 5DAFBE7A
 P 9250 3550
@@
 $EndComp
 $Comp
-L elements:Конденсатор_керамический C?
+L mag-rescue:Конденсатор_керамический-elements C?
 U 1 1 5DAC0C48
 P 8500 3550
@@
 	6000 3900 5750 3900
 $Comp
-L elements:Конденсатор_керамический C?
+L mag-rescue:Конденсатор_керамический-elements C?
 U 1 1 5DAEAF30
 P 5000 4050
@@
 $EndComp
 $Comp
-L elements:Резистор_0,065Вт R?
+L mag-rescue:Резистор_0,065Вт-elements R?
 U 1 1 5DAD5F00
 P 8000 4650
@@
 $EndComp
 $Comp
-L elements:Резистор_0,065Вт R?
+L mag-rescue:Резистор_0,065Вт-elements R?
 U 1 1 5DAD5865
 P 8000 3800
@@
 $EndComp
 $Comp
-L elements:Чип-индуктивность L1
+L mag-rescue:Чип-индуктивность-elements L1
 U 1 1 5DABFCBC
 P 6700 3250
@@
 $EndComp
 $Comp
-L elements:Диод_шоттки VD6
+L mag-rescue:Диод_шоттки-elements VD6
 U 1 1 5DABC3D5
 P 7500 3250
@@
 $EndComp
 $Comp
-L elements:Микросхема_DCDC_step_UP_LM2703 G2
+L mag-rescue:Микросхема_DCDC_step_UP_LM2703-elements G2
 U 1 1 5DABB5AB
 P 6200 3750
@@
 	7950 2000 7950 2200
 $Comp
-L elements:Конденсатор_керамический C?
+L mag-rescue:Конденсатор_керамический-elements C?
 U 1 1 5DA73B6B
 P 7950 2250
@@
 	9200 2000 9200 2200
 $Comp
-L elements:Конденсатор_керамический C?
+L mag-rescue:Конденсатор_керамический-elements C?
 U 1 1 5DA73764
 P 9200 2250
@@
 3V_out
 $Comp
-L elements:стабилизатор_нерегулируемый_XC6206P302MR G1
+L mag-rescue:стабилизатор_нерегулируемый_XC6206P302MR-elements G1
 U 1 1 5DA41F3D
 P 8250 2000
@@
 Bat_out+
 $Comp
-L elements:кнопка K?
+L mag-rescue:кнопка-elements K?
 U 1 1 5D96CFE8
 P 3500 6250
@@
 $EndComp
 $Comp
-L elements:Резистор_0,065Вт R?
+L mag-rescue:Резистор_0,065Вт-elements R?
 U 1 1 5D96E506
 P 2950 5300
@@
 $EndComp
 $Comp
-L elements:Транзистор_полевой_P-канал(IRLML2246TRPBF) VT1
+L mag-rescue:Транзистор_полевой_P-канал(IRLML2246TRPBF)-elements VT1
 U 1 1 5D976703
 P 3750 5550
@@
 pwr_on_off
 $Comp
-L elements:Резистор_0,065Вт R?
+L mag-rescue:Резистор_0,065Вт-elements R?
 U 1 1 5D9A0DAF
 P 8300 6000
