File: mag/mag.sch (KiCad schematic (older format))
At the start: 28 parts, among them K1 кнопка_FSMSM, K2 кнопка_FSMSM, X1 Клеммник_х2

Commit message: тестовая прошивка, замечания по плате
тестовая прошивка - обмен по usb-uart
замечания по плате - добавлены пометки для изсправления в следующих версиях
Parts:
- X1: symbol elements:Клеммник_х2 -> mag-rescue:Клеммник_х2-elements
Other:
- note added: "убрать ключ напротив MOSI"
Changed lines of the file:
@@
 	4550 9900 4550 10000
 $Comp
-L elements:Клеммник_х2 X1
+L mag-rescue:Клеммник_х2-elements X1
 U 1 1 5DB281F4
 P 2500 2750
@@
 Wire Wire Line
 	10500 1750 10750 1750
+Text Notes 7700 8200 0    50   ~ 0
+убрать ключ напротив MOSI
 $EndSCHEMATC

Commit message: библиотека bmp180, замечания к схеме
Parts:
- C1, C2, C3, C4, C5: symbol elements:Конденсатор_керамический -> mag-rescue:Конденсатор_керамический-elements
- DD1: symbol elements:ATmega8A-AU -> mag-rescue:ATmega8A-AU-elements
- DD2, DD3, DD4, DD5: symbol elements:D-triger_8bit -> mag-rescue:D-triger_8bit-elements
- HL1: symbol elements:display_EDS803_EDS805 -> mag-rescue:display_EDS803_EDS805-elements
- HL2: symbol elements:Розетка_PBS4 -> mag-rescue:Розетка_PBS4-elements
- K1, K2: symbol elements:кнопка -> mag-rescue:кнопка-elements
- R1, R15, R16, R17, R18, R19, R2, R20, R3, R4, R5: symbol elements:Резистор_0,065Вт -> mag-rescue:Резистор_0,065Вт-elements
- XP3: symbol elements:Вилка_PLD6_ПРОГ -> mag-rescue:Вилка_PLD6_ПРОГ-elements
- XP4: symbol elements:Вилка_PLS4 -> mag-rescue:Вилка_PLS4-elements
Other:
- note added: "замена на 100 Ом"
Changed lines of the file:
@@
 EESchema Schematic File Version 4
 LIBS:mag-cache
-EELAYER 29 0
+EELAYER 30 0
 EELAYER END
 $Descr A3 16535 11693
@@
 $EndDescr
 $Comp
-L elements:ATmega8A-AU DD1
+L mag-rescue:ATmega8A-AU-elements DD1
 U 1 1 5CE45047
 P 2400 6500
@@
 $EndComp
 $Comp
-L elements:Резистор_0,065Вт R2
+L mag-rescue:Резистор_0,065Вт-elements R2
 U 1 1 5CE45133
 P 2950 5150
@@
 $EndComp
 $Comp
-L elements:Резистор_0,065Вт R1
+L mag-rescue:Резистор_0,065Вт-elements R1
 U 1 1 5CE451D9
 P 2250 5150
@@
 SCL
 $Comp
-L elements:Вилка_PLD6_ПРОГ XP3
+L mag-rescue:Вилка_PLD6_ПРОГ-elements XP3
 U 1 1 5CE4524F
 P 7750 7650
@@
 RES
 $Comp
-L elements:D-triger_8bit DD2
+L mag-rescue:D-triger_8bit-elements DD2
 U 1 1 5CE49B21
 P 7400 4500
@@
 	12500 1800 12200 1800
 $Comp
-L elements:Розетка_PBS4 HL2
+L mag-rescue:Розетка_PBS4-elements HL2
 U 1 1 5CE597ED
 P 11700 1400
@@
 $EndComp
 $Comp
-L elements:D-triger_8bit DD3
+L mag-rescue:D-triger_8bit-elements DD3
 U 1 1 5CE59956
 P 9600 4500
@@
 	9400 4500 9100 4500
 $Comp
-L elements:D-triger_8bit DD4
+L mag-rescue:D-triger_8bit-elements DD4
 U 1 1 5CE5ACE2
 P 11800 4500
@@
 	11600 4500 11300 4500
 $Comp
-L elements:D-triger_8bit DD5
+L mag-rescue:D-triger_8bit-elements DD5
 U 1 1 5CE5ACFE
 P 14000 4500
@@
 Display
 $Comp
-L elements:display_EDS803_EDS805 HL1
+L mag-rescue:display_EDS803_EDS805-elements HL1
 U 1 1 5CEAE07F
 P 13750 1000
@@
 	8400 5850 8100 5850
 $Comp
-L elements:кнопка K1
+L mag-rescue:кнопка-elements K1
 U 1 1 5D0AA259
 P 2050 8800
@@
 $EndComp
 $Comp
-L elements:кнопка K2
+L mag-rescue:кнопка-elements K2
 U 1 1 5D0ADEEF
 P 2050 9250
@@
 	4650 6800 4350 6800
 $Comp
-L elements:Резистор_0,065Вт R3
+L mag-rescue:Резистор_0,065Вт-elements R3
 U 1 1 5D14357F
 P 3600 5150
@@
 	4350 7900 4650 7900
 $Comp
-L elements:Резистор_0,065Вт R4
+L mag-rescue:Резистор_0,065Вт-elements R4
 U 1 1 5D2DD9FC
 P 4400 4700
@@
 $EndComp
 $Comp
-L elements:Резистор_0,065Вт R5
+L mag-rescue:Резистор_0,065Вт-elements R5
 U 1 1 5D2E0229
 P 4400 5400
@@
 $EndSheet
 $Comp
-L elements:Вилка_PLS4 XP4
+L mag-rescue:Вилка_PLS4-elements XP4
 U 1 1 5D953B57
 P 2000 1650
@@
 	2500 1750 3000 1750
 $Comp
-L elements:Конденсатор_керамический C1
+L mag-rescue:Конденсатор_керамический-elements C1
 U 1 1 5DA4B9C4
 P 1500 10150
@@
 $EndComp
 $Comp
-L elements:Конденсатор_керамический C2
+L mag-rescue:Конденсатор_керамический-elements C2
 U 1 1 5DA4B9CC
 P 2250 10150
@@
 $EndComp
 $Comp
-L elements:Конденсатор_керамический C3
+L mag-rescue:Конденсатор_керамический-elements C3
 U 1 1 5DA4B9D4
 P 3000 10150
@@
 $EndComp
 $Comp
-L elements:Конденсатор_керамический C4
+L mag-rescue:Конденсатор_керамический-elements C4
 U 1 1 5DA4B9DC
 P 3750 10150
@@
 Connection ~ 3000 10350
 $Comp
-L elements:Конденсатор_керамический C5
+L mag-rescue:Конденсатор_керамический-elements C5
 U 1 1 5DA4B9FC
 P 4550 10150
@@
 SCL
 $Comp
-L elements:Резистор_0,065Вт R16
+L mag-rescue:Резистор_0,065Вт-elements R16
 U 1 1 5D9E1F2D
 P 1750 5150
@@
 $EndComp
 $Comp
-L elements:Резистор_0,065Вт R15
+L mag-rescue:Резистор_0,065Вт-elements R15
 U 1 1 5D9E20AE
 P 1250 5150
@@
 VCC_bat
 $Comp
-L elements:Резистор_0,065Вт R17
+L mag-rescue:Резистор_0,065Вт-elements R17
 U 1 1 5DA74EF5
 P 5350 10000
@@
 NoConn ~ 8200 7500
 $Comp
-L elements:Резистор_0,065Вт R20
+L mag-rescue:Резистор_0,065Вт-elements R20
 U 1 1 5DBE5539
 P 9050 7650
@@
 	8200 7650 8750 7650
 $Comp
-L elements:Резистор_0,065Вт R19
+L mag-rescue:Резистор_0,065Вт-elements R19
 U 1 1 5DC136FC
 P 6450 7650
@@
 $EndComp
 $Comp
-L elements:Резистор_0,065Вт R18
+L mag-rescue:Резистор_0,065Вт-elements R18
 U 1 1 5DC14E63
 P 6450 7250
@@
 Text Notes 7700 8200 0    50   ~ 0
 убрать ключ напротив MOSI
+Text Notes 5350 10300 0    50   ~ 0
+замена на 100 Ом
 $EndSCHEMATC

Commit message: проверка исправности LCD дисплея
обнаружена проблема с питанием контроллера: p-канальный транзистор через что-то утекает и сам открывается
Other:
- note added: "SDA и SCL подтянуть к 3В, а не батарее"
Changed lines of the file:
@@
 Text Notes 5350 10300 0    50   ~ 0
 замена на 100 Ом
+Text Notes 1950 4450 0    50   ~ 0
+SDA и SCL подтянуть к 3В, а не батарее
 $EndSCHEMATC

Commit message: доопределен адрес дисплея, добавлена функция инициализации дисплея
Other:
- note added: "Display\nadres: 0x3С (0011 110b)"
- note removed: "Display"
Changed lines of the file:
@@
 Wire Wire Line
 	13800 4500 13500 4500
-Text Notes 11750 2000 0    50   ~ 0
-Display
 $Comp
 L mag-rescue:display_EDS803_EDS805-elements HL1
@@
 Text Notes 1950 4450 0    50   ~ 0
 SDA и SCL подтянуть к 3В, а не батарее
+Text Notes 11600 2100 0    50   ~ 0
+Display\nadres: 0x3С (0011 110b)
 $EndSCHEMATC

Commit message: инициирован переезд на ESP32
Parts:
- removed C1, C2, C3, C4, C5: Конденсатор_керамический, N_RLC:Конденсатор_SMD_0603, symbol mag-rescue:Конденсатор_керамический-elements
- removed DD1: ATmega328, N_DD:микросхема_ATMEGA-8-161AU, symbol mag-rescue:ATmega8A-AU-elements
- removed DD2, DD3, DD4, DD5: D-triger_74VHC573MTC, N_DD:SSOP-20, symbol mag-rescue:D-triger_8bit-elements
- removed HL1: display_EDS803_EDS805, N_VD_HL:display_EDS803_805, symbol mag-rescue:display_EDS803_EDS805-elements
- removed HL2: oled_0.91_128x32, N_VD_HL:oled_0.91_128x32, symbol mag-rescue:Розетка_PBS4-elements
- removed K1, K2: кнопка_FSMSM, N_X:Кнопка_FSMSM, symbol mag-rescue:кнопка-elements
- removed R1, R15, R16, R17, R18, R19, R2, R20, R3, R4, R5: Резистор_0,065Вт, N_RLC:Конденсатор_SMD_0603, symbol mag-rescue:Резистор_0,065Вт-elements
- removed X1: Клеммник_х2, N_X:Вилка_PLS2_вертикальная, symbol mag-rescue:Клеммник_х2-elements
- removed XP3: Вилка_PLD6_ПРОГ, N_X:Вилка_PLD6_вертикальная, symbol mag-rescue:Вилка_PLD6_ПРОГ-elements
- removed XP4: USB_female, N_X:Вилка_PLS4_вертикальная, symbol mag-rescue:Вилка_PLS4-elements
- added A1: модуль_esp32_wroom_32_SMD_noSD, N_A:ESP32_WROOM32_pnp_noSD, symbol modules:модуль_esp32_wroom_32_SMD_noSD
- added C1, C2: Конденсатор_керамический, N_RLC:Конденсатор_SMD_IEC_0805, symbol elements:Конденсатор_керамический
- added C10, C11, C13, C4: Конденсатор*0,1мкФ*25В*0603, N_RLC:Конденсатор_SMD_IEC_0603, symbol eo-engine:Конденсатор*0,1мкФ*25В*0603
- added C12: Конденсатор*10мкФ*16В*0805, N_RLC:Конденсатор_SMD_IEC_0805, symbol eo-engine:Конденсатор*10мкФ*16В*0805
- added C3, C5: Конденсатор_керамический, N_RLC:Конденсатор_SMD_0603_pnp, symbol elements:Конденсатор_керамический
- added C6, C7, C8, C9: Конденсатор_керамический, N_RLC:Конденсатор_SMD_0603, symbol mag-rescue:Конденсатор_керамический-elements
- added D1: LOGO, N_ICO:ni_10x10, symbol elements:LOGO
- added DA1: ОУ_LM358DT, MOTOR_IMPORT_OTK:SO-8, symbol MOTOR_2020_import:ОУ_LM358DT
- added DA2: ОУ_LMV321ILT, N_G:SOT-23-5_pnp, symbol elements_2020:ОУ_LMV321ILT
- added DD1: Микросхема_заряда_MCP73831T-2ACI_OT, N_G:SOT-23-5_pnp, symbol elements_2020:Микросхема_заряда_MCP73831T-2ACI_OT
- added DD2: LIS3DH, N_DD:акселерометр_LIS3DH, symbol mag-rescue:LIS3DH-elements
- added DD3: Преобразователь_CP2102(USB-UART), N_DD:Микросхема_CP2102, symbol mag-rescue:Преобразователь_CP2102(USB-UART)-elements
- added DD4: Датчик_bmp180, N_DD:BMP180, symbol mag-rescue:Датчик_bmp180-elements
- added FU1: Предохранитель_MF-MSMF030, N_RLC:Предохранитель_SMD_1812, symbol elements:Предохранитель
- added G1: ИОП_LM4040BIM3-2.5_NOPB, N_VD_HL:Транзистор_IRLML6344TR_SOT-23, symbol elements_2020:ИОП_LM4040BIM3-2.5_NOPB
- added HL1: Светодиод_сдвоенный_KPB-3025SURKCGKC, N_VD_HL:Светодиод_SMD_m3025, symbol elements_2020:Светодиод_сдвоенный_KPB-3025SURKCGKC
- added HL2: TFT-дисплей_ST7735_ILI9341, N_VD_HL:TFT_2.8_INCH, symbol elements_2020:TFT-дисплей_ST7735_ILI9341
- added K1, K2: Кнопка_KLS7-TS5401-1.35-250-T, N_X:Кнопка_KLS7-TS5401, symbol elements_2020:Кнопка_KLS7-TS5401-1.35-250-T
- added R1, R11, R12, R13, R14, R15, R17, R18, R2, R21, R23, R24, R25, R3, R8, R9: Резистор_0,065Вт, N_RLC:Резистор_SMD_0603_0,065_Вт, symbol elements:Резистор_0,065Вт
- added R10, R16, R22, R29, R4, R6: Резистор*1кОм*0603, N_RLC:Резистор_SMD_0603_0,065_Вт_pnp, symbol eo-engine:Резистор*10кОм*0603
- added R19: Резистор*2,4кОм*0603, N_RLC:Резистор_SMD_0603_0,065_Вт_pnp, symbol eo-engine:Резистор*10кОм*0603
- added R20, R5: Резистор*10кОм*0603, N_RLC:Резистор_SMD_0603_0,065_Вт_pnp, symbol eo-engine:Резистор*10кОм*0603
- added R26, R27, R28: Резистор_0,065Вт, N_RLC:Конденсатор_SMD_0603, symbol mag-rescue:Резистор_0,065Вт-elements
- added R7: Резистор*1Ом*0603, N_RLC:Резистор_SMD_0603_0,065_Вт_pnp, symbol eo-engine:Резистор*10кОм*0603
- added VD1: Набор_диодов_2Д803АС9, MOTOR_VD_VT_HL:Корпус_КТ-46, symbol MOTOR_2020_components:Набор_диодов_2Д803АС9
- added VD2, VD3, VD5: Стабилитрон*3,3В*SOD80, N_VD_HL:SOD-80, symbol eo-engine:Стабилитрон*3,3В*SOD80
- added VD4: Диоды_шоттки_BAR43CFILM, N_VD_HL:Транзистор_IRLML6344TR_SOT-23, symbol elements_2020:Диоды_шоттки_BAR43CFILM
- added VD6: Стабилитрон_BZV55-C3V9, N_VD_HL:SOD-80, symbol elements_2020:Стабилитрон_1N5352BRLG_вертикальный
- added VT1, VT3, VT7: Транзистор_полевой_P-канал(IRLML2246TRPBF), N_VD_HL:Транзистор_IRLML6344TR_SOT-23, symbol elements:Транзистор_полевой_P-канал(IRLML2246TRPBF)
- added VT2, VT6: Транзистор*pnp*0,5А*45В*SOT23, N_VD_HL:Корпус_КТ-46, symbol eo-engine:Транзистор*pnp*0,5А*45В*SOT23
- added VT4: Транзистор_полевой_N-IRLML6344TR, N_VD_HL:Транзистор_IRLML6344TR_SOT-23, symbol elements:Транзистор_полевой_N-IRLML6344TR
- added VT5: Транзистор*npn*0,5А*45В*SOT23, N_VD_HL:Корпус_КТ-46, symbol eo-engine:Транзистор*npn*0,5А*45В*SOT23
- added X1, X2, X3, X4: отверстие_под_пайку, N_X:ОтверстиеD1.2, symbol elements:отверстие_под_пайку
- added XS1: UBS-type-C-105450-0101&упрощенная, N_X:usb-type-c, symbol elements_2020:UBS-type-C-105450-0101&упрощенная
Connections:
- net labels added: #метка-3V3, #метка-5V, #метка-GND, 3V3, AN.2V5.REF, AN.BAT.MEASURE, BAT.CHARGE, BAT.IN, BAT.LOAD, BOOT, BOOT-UART-RX, BOOT-UART-TX, BUTT.TURN, CHARGE.MODE, CUR-DIRECT, CUR-SENS, D+, D-, EXT.BUTT, GND, GND-IN, I2C_SCL, I2C_SDA, MISO, MOSI, REF-0V1, REF-3V3, RESET, SCK, SELF.TURN, TFT-CS, TFT-DC, TFT-LED, TFT-RES, U.FB, U.IN, U.PROTECT, UIN, USB_pwr, USB_pwr_gnd, VCCbat, VOL-DIRECT, VOL-SENS, max0.3A, max4V1, vcc
- net labels removed: 5V, ADC6, AREF, Out11, Out12, Out13, Out14, Out15, Out16, Out17, Out18, Out21, Out22, Out23, Out24, Out25, Out26, Out27, Out28, Out31, Out32, Out33, Out34, Out35, Out36, Out37, Out38, Out41, Out42, Out43, Out44, Out45, Out46, Out47, Out48, PB0, PB1, PB2, PB3_MOSI, PB4_MISO, PB5_SCK, PB6, PB7, PC0, PC1, PC2, PC3, PD3, PD4, PD5, PD6, PD7, RES, VCC_bat
- wire segments 236 -> 319
- no-connect marks 8 -> 18
Other:
- note added: "-нажатие кнопки открывает транзистор питания\n-на линии SELF.TURN МК должен выставить высокий уровень для самоподхвата\n-на лии BUTT.TURN МК в режиме PULL-UP видит состояние кнопки включения"
- note added: "1) кнопка питания от АБ - удержание, как на включение, так и на выключение\n2)+ ограничение входного тока на уровне 0,3А\n3)+ ограничение напряжения за источником тока на уровне 4,1В\n4) стабилизация напряжения от АБ на уровне 3,3В, ток не менее 1А\n5)+ защита от входной переполюсовки диодом\n6) светодиод завершения заряда"
- note added: "LP383450, Аккумулятор литий-полимерный (Li-Pol) 800мАч 3.7В, с защитой\n34 х 50 мм"
- note added: "~~300 мА"
- note added: "Акселерометр\nadres: 0x19 (0011 001b)"
- note added: "Альтиметр\nadres: 0x77 (1110 111b)"
- note added: "СХЕМА СБРОСА"
- note added: "включение питания с самоподхватом"
- note added: "защита от переполюсовки"
- note removed: "Display\nadres: 0x3С (0011 110b)"
- note removed: "SDA и SCL подтянуть к 3В, а не батарее"
- note removed: "USB type C"
- note removed: "Информация"
- note removed: "Подключение аккумулятора"
- note removed: "Режим/Работа"
- note removed: "замена на 100 Ом"
- note removed: "убрать ключ напротив MOSI"

Commit message: подготовлена схема заряда АБ, начата схема питания МК
Parts:
- added C14: Конденсатор*10мкФ*16В*0805, N_RLC:Конденсатор_SMD_IEC_0805, symbol eo-engine:Конденсатор*10мкФ*16В*0805
- added G2: Микросхема*LDO*IN8V*OUT3V3*1,2A*SOT-223, N_VD_HL:Транзистор_NPN_SOT223_pnp, symbol eo-engine:Микросхема*LDO*IN8V*OUT3V3*1,2A*SOT-223
Connections:
- net 3V3: now also C14.1, G2.2 (OUT(2V5)), G2.4 (OUT(2V5))
- net GND: now also C12.2, C14.2, G2.1 (GND)
- net at C12.1: now also G2.3 (IN)
Other:
- note added: "совместить линейный стабилизатор и включение по кнопке"
- moved on the sheet: C12
Changed lines of the file:
@@
 L eo-engine:#метка-3V3 #3V1
 U 1 1 644DD9E6
-P 16150 3300
-F 0 "#3V1" H 16150 3250 50  0001 C CNN
-F 1 "#метка-3V3" H 16100 3150 50  0001 C CNN
-F 2 "" H 16150 3300 50  0001 C CNN
-F 3 "" H 16150 3300 50  0001 C CNN
-	1    16150 3300
+P 21000 1750
+F 0 "#3V1" H 21000 1700 50  0001 C CNN
+F 1 "#метка-3V3" H 20950 1600 50  0001 C CNN
+F 2 "" H 21000 1750 50  0001 C CNN
+F 3 "" H 21000 1750 50  0001 C CNN
+	1    21000 1750
 	1    0    0    -1
 $EndComp
@@
 L eo-engine:#метка-GND #GND2
 U 1 1 650E835F
-P 15250 2500
-F 0 "#GND2" H 15250 2550 50  0001 C CNN
-F 1 "#метка-GND" H 15300 2650 50  0001 C CNN
-F 2 "" H 15250 2500 50  0001 C CNN
-F 3 "" H 15250 2500 50  0001 C CNN
-	1    15250 2500
+P 16500 2500
+F 0 "#GND2" H 16500 2550 50  0001 C CNN
+F 1 "#метка-GND" H 16550 2650 50  0001 C CNN
+F 2 "" H 16500 2500 50  0001 C CNN
+F 3 "" H 16500 2500 50  0001 C CNN
+	1    16500 2500
 	-1   0    0    -1
 $EndComp
-Wire Wire Line
-	15000 2500 15250 2500
 Wire Wire Line
 	13250 6000 15500 6000
@@
 L eo-engine:Конденсатор*10мкФ*16В*0805 C12
 U 1 1 652ACB3B
-P 8000 -750
-F 0 "C12" H 8184 -866 138 0000 L CNN
-F 1 "Конденсатор*10мкФ*16В*0805" H 7850 -500 50  0001 C CNN
-F 2 "N_RLC:Конденсатор_SMD_IEC_0805" H 7950 -600 50  0001 C CNN
-F 3 "" H 8000 -750 50  0001 C CNN
-F 4 "10мкФ 16В" H 8184 -1089 138 0000 L CNN "INFO"
-F 5 "https://www.terraelectronica.ru/product/863492" H 7950 -600 50  0001 C CNN "LINK"
-F 6 "0,86" H 8000 -750 50  0001 C CNN "COST"
-	1    8000 -750
+P 16500 1850
+F 0 "C12" H 16684 1734 138 0000 L CNN
+F 1 "Конденсатор*10мкФ*16В*0805" H 16350 2100 50  0001 C CNN
+F 2 "N_RLC:Конденсатор_SMD_IEC_0805" H 16450 2000 50  0001 C CNN
+F 3 "" H 16500 1850 50  0001 C CNN
+F 4 "10мкФ 16В" H 16684 1511 138 0000 L CNN "INFO"
+F 5 "https://www.terraelectronica.ru/product/863492" H 16450 2000 50  0001 C CNN "LINK"
+F 6 "0,86" H 16500 1850 50  0001 C CNN "COST"
+	1    16500 1850
 	1    0    0    -1
 $EndComp
@@
 Wire Wire Line
 	13250 1750 15000 1750
+Connection ~ 13250 1750
+$Comp
+L eo-engine:Микросхема*LDO*IN8V*OUT3V3*1,2A*SOT-223 G2
+U 1 1 6421A54A
+P 18500 1750
+F 0 "G2" H 19500 2100 138 0000 C CNN
+F 1 "Микросхема*LDO*IN8V*OUT3V3*1,2A*SOT-223" H 19100 700 50  0001 C CNN
+F 2 "N_VD_HL:Транзистор_NPN_SOT223_pnp" H 18500 1950 50  0001 C CNN
+F 3 "https://static.chipdip.ru/lib/529/DOC010529765.pdf" H 18500 1950 50  0001 C CNN
+F 4 "https://www.chipdip.ru/product/ldl1117s33r-stm" H 18500 1750 50  0001 C CNN "LINK"
+F 5 "LDO 3V3" H 19500 1100 138 0000 C CNN "INFO"
+	1    18500 1750
+	1    0    0    -1
+$EndComp
+Wire Wire Line
+	20500 1750 21000 1750
+Wire Wire Line
+	20500 2050 21000 2050
+Wire Wire Line
+	21000 2050 21000 1750
+Connection ~ 21000 1750
+$Comp
+L eo-engine:Конденсатор*10мкФ*16В*0805 C14
+U 1 1 642AEDB7
+P 21000 2250
+F 0 "C14" H 21184 2134 138 0000 L CNN
+F 1 "Конденсатор*10мкФ*16В*0805" H 20850 2500 50  0001 C CNN
+F 2 "N_RLC:Конденсатор_SMD_IEC_0805" H 20950 2400 50  0001 C CNN
+F 3 "" H 21000 2250 50  0001 C CNN
+F 4 "10мкФ 16В" H 21184 1911 138 0000 L CNN "INFO"
+F 5 "https://www.terraelectronica.ru/product/863492" H 20950 2400 50  0001 C CNN "LINK"
+F 6 "0,86" H 21000 2250 50  0001 C CNN "COST"
+	1    21000 2250
+	1    0    0    -1
+$EndComp
+Wire Wire Line
+	16000 1750 16500 1750
+Wire Wire Line
+	16500 2500 16500 2350
+Connection ~ 16500 2500
+Wire Wire Line
+	16500 1850 16500 1750
+Connection ~ 16500 1750
+Wire Wire Line
+	16500 1750 18500 1750
+Wire Wire Line
+	16500 2500 18250 2500
+Wire Wire Line
+	18250 2500 18250 2050
+Wire Wire Line
+	18250 2050 18500 2050
+$Comp
+L eo-engine:#метка-GND #GND3
+U 1 1 6435EB5B
+P 21000 3000
+F 0 "#GND3" H 21000 3050 50  0001 C CNN
+F 1 "#метка-GND" H 21050 3150 50  0001 C CNN
+F 2 "" H 21000 3000 50  0001 C CNN
+F 3 "" H 21000 3000 50  0001 C CNN
+	1    21000 3000
+	-1   0    0    -1
+$EndComp
+Wire Wire Line
+	21000 2050 21000 2250
+Connection ~ 21000 2050
+Wire Wire Line
+	21000 2750 21000 3000
+Text Notes 15500 4000 0    138  ~ 0
+совместить линейный стабилизатор и включение по кнопке
+Wire Wire Line
+	15000 2500 16500 2500
 Wire Bus Line
 	3000 2850 3000 6400
-Connection ~ 13250 1750
 $EndSCHEMATC

Commit message: подготовлена схема включения 3,3В, не установлен источник 2,5В
Parts:
- removed C1, C2: Конденсатор_керамический, N_RLC:Конденсатор_SMD_IEC_0805, symbol elements:Конденсатор_керамический
- removed DD1: Микросхема_заряда_MCP73831T-2ACI_OT, N_G:SOT-23-5_pnp, symbol elements_2020:Микросхема_заряда_MCP73831T-2ACI_OT
- removed FU1: Предохранитель_MF-MSMF030, N_RLC:Предохранитель_SMD_1812, symbol elements:Предохранитель
- removed G2: Микросхема*LDO*IN8V*OUT3V3*1,2A*SOT-223, N_VD_HL:Транзистор_NPN_SOT223_pnp, symbol eo-engine:Микросхема*LDO*IN8V*OUT3V3*1,2A*SOT-223
- removed R1, R2, R3, R8: Резистор_0,065Вт, N_RLC:Резистор_SMD_0603_0,065_Вт, symbol elements:Резистор_0,065Вт
- removed VT1: Транзистор_полевой_P-канал(IRLML2246TRPBF), N_VD_HL:Транзистор_IRLML6344TR_SOT-23, symbol elements:Транзистор_полевой_P-канал(IRLML2246TRPBF)
- added C15, C16: Конденсатор*0,1мкФ*25В*0603, N_RLC:Конденсатор_SMD_IEC_0603, symbol eo-engine:Конденсатор*0,1мкФ*25В*0603
- added DA3: ОУ_LM358DT, MOTOR_IMPORT_OTK:SO-8, symbol MOTOR_2020_import:ОУ_LM358DT
- added R30: Резистор*10кОм*0603, N_RLC:Резистор_SMD_0603_0,065_Вт_pnp, symbol eo-engine:Резистор*10кОм*0603
- added R31, R32, R33: Резистор*1кОм*0603, N_RLC:Резистор_SMD_0603_0,065_Вт_pnp, symbol eo-engine:Резистор*10кОм*0603
- added VD7: Стабилитрон*3,3В*SOD80, N_VD_HL:SOD-80, symbol eo-engine:Стабилитрон*3,3В*SOD80
- added VT10, VT9: Транзистор*pnp*0,5А*45В*SOT23, N_VD_HL:Корпус_КТ-46, symbol eo-engine:Транзистор*pnp*0,5А*45В*SOT23
- added VT8: Транзистор_полевой_N-канальный_КП526А9, MOTOR_VD_VT_HL:Корпус_КТ-46, symbol elements_2020:Транзистор_полевой_N-канальный_КП526А9
Connections:
- net 3V3: now also DA3.3, VT10.3, VT9.3
- net GND: now also C16.2, R30.1, VT8.2; no longer K1.3, K1.4
- net REF-3V3: now also C16.1, DA3.2
- net max4V1: now also C12.1, K1.3, K1.4, C15.1, DA3.8 (VCC), VT10.2, VT9.2
- net at K1.1, K1.2: now also R33.1; no longer R11.1, R9.1
- net BAT.CHARGE: no longer names the net of R12.1, VT3.2
- new net: R11.1, R9.1
- new net: R32.1, VT10.1
- new net: R31.1, VT9.1
- new net: R31.2, R32.2, VD7.2
- new net: R30.2, R33.2, VT8.1
- new net COM: C15.2, DA3.4 (GND), VT8.3
- new net LDO-DIRECT: DA3.1, VD7.1
Other:
- note added: "питание 2,5В для i2c датчиков"
- note removed: "~~300 мА"
- note removed: "защита от переполюсовки"
- note removed: "совместить линейный стабилизатор и включение по кнопке"
- moved on the sheet: A1, C12, C14, C3, C5, DA2, G1, K1, K2, R11, R12, R13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
