File: mag/mag.sch (KiCad schematic (older format))
At the start: 77 parts, among them K1 Кнопка_KLS7-TS5401-1.35-250-T, K2 Кнопка_KLS7-TS5401-1.35-250-T, X1 отверстие_под_пайку, X2 отверстие_под_пайку, X3 отверстие_под_пайку, X4 отверстие_под_пайку

Commit message: вынесен, но не подключен LDO на 2,5В
Parts:
- added G2: Микросхема*LDO*IN8V*OUT2V5*1,2A*SOT-223, N_VD_HL:Транзистор_NPN_SOT223_pnp, symbol eo-engine:Микросхема*LDO*IN8V*OUT3V3*1,2A*SOT-223
Connections:
- no-connect marks 18 -> 21
Other:
- moved on the sheet: C15, K1, R30, R33, VT8
Changed lines of the file:
@@
 L elements_2020:Кнопка_KLS7-TS5401-1.35-250-T K1
 U 1 1 614C6E2B
-P 21550 6850
-F 0 "K1" V 21750 7050 50  0000 R CNN
-F 1 "Кнопка_KLS7-TS5401-1.35-250-T" V 21504 6800 50  0001 R CNN
-F 2 "N_X:Кнопка_KLS7-TS5401" H 21550 6875 50  0001 C CNN
-F 3 "" H 21550 6875 50  0001 C CNN
-	1    21550 6850
+P 21550 7150
+F 0 "K1" V 21750 7350 50  0000 R CNN
+F 1 "Кнопка_KLS7-TS5401-1.35-250-T" V 21504 7100 50  0001 R CNN
+F 2 "N_X:Кнопка_KLS7-TS5401" H 21550 7175 50  0001 C CNN
+F 3 "" H 21550 7175 50  0001 C CNN
+	1    21550 7150
 	0    -1   -1   0
 $EndComp
@@
 L elements_2020:Транзистор_полевой_N-канальный_КП526А9 VT8
 U 1 1 64098EFF
-P 19550 6500
-F 0 "VT8" H 19700 7100 138 0000 C CNN
-F 1 "Транзистор_полевой_N-канальный_КП526А9" H 19700 7001 60  0001 C CNN
-F 2 "MOTOR_VD_VT_HL:Корпус_КТ-46" H 19625 7175 60  0001 C CNN
-F 3 "" H 19550 6500 60  0001 C CNN
-F 4 "https://www.chipdip.ru/product/kp526a9" H 19575 7350 50  0001 C CNN "LINK"
-F 5 "1,25А 30В" H 20700 6650 138 0000 C CNN "INFO"
-	1    19550 6500
+P 19550 6800
+F 0 "VT8" H 19700 7400 138 0000 C CNN
+F 1 "Транзистор_полевой_N-канальный_КП526А9" H 19700 7301 60  0001 C CNN
+F 2 "MOTOR_VD_VT_HL:Корпус_КТ-46" H 19625 7475 60  0001 C CNN
+F 3 "" H 19550 6800 60  0001 C CNN
+F 4 "https://www.chipdip.ru/product/kp526a9" H 19575 7650 50  0001 C CNN "LINK"
+F 5 "1,25А 30В" H 20700 6950 138 0000 C CNN "INFO"
+	1    19550 6800
 	-1   0    0    -1
 $EndComp
 Wire Wire Line
-	19000 6200 18500 6200
+	19000 6500 18500 6500
 Wire Wire Line
 	18500 5600 19000 5600
@@
 L eo-engine:#метка-GND #GND4
 U 1 1 640BC4E8
-P 18750 7200
-F 0 "#GND4" H 18750 7250 50  0001 C CNN
-F 1 "#метка-GND" H 18800 7350 50  0001 C CNN
-F 2 "" H 18750 7200 50  0001 C CNN
-F 3 "" H 18750 7200 50  0001 C CNN
-	1    18750 7200
-	1    0    0    -1
-$EndComp
-Wire Wire Line
-	18750 7200 18750 7000
-Wire Wire Line
-	18750 6500 19000 6500
+P 18750 7500
+F 0 "#GND4" H 18750 7550 50  0001 C CNN
+F 1 "#метка-GND" H 18800 7650 50  0001 C CNN
+F 2 "" H 18750 7500 50  0001 C CNN
+F 3 "" H 18750 7500 50  0001 C CNN
+	1    18750 7500
+	1    0    0    -1
+$EndComp
+Wire Wire Line
+	18750 7500 18750 7300
+Wire Wire Line
+	18750 6800 19000 6800
 $Comp
 L eo-engine:Резистор*10кОм*0603 R30
 U 1 1 640F8807
-P 19100 7000
-F 0 "R30" H 19400 6800 138 0000 C CNN
-F 1 "Резистор*10кОм*0603" H 19100 7600 50  0001 C CNN
-F 2 "N_RLC:Резистор_SMD_0603_0,065_Вт_pnp" H 19200 7500 50  0001 C CNN
-F 3 "" V 19100 7000 50  0001 C CNN
-F 4 "10к" H 19400 7250 138 0000 C CNN "INFO"
-	1    19100 7000
+P 19100 7300
+F 0 "R30" H 19400 7100 138 0000 C CNN
+F 1 "Резистор*10кОм*0603" H 19100 7900 50  0001 C CNN
+F 2 "N_RLC:Резистор_SMD_0603_0,065_Вт_pnp" H 19200 7800 50  0001 C CNN
+F 3 "" V 19100 7300 50  0001 C CNN
+F 4 "10к" H 19400 7550 138 0000 C CNN "INFO"
+	1    19100 7300
 	1    0    0    1
 $EndComp
 Wire Wire Line
-	18750 7000 19100 7000
-Connection ~ 18750 7000
-Wire Wire Line
-	18750 7000 18750 6500
+	18750 7300 19100 7300
+Connection ~ 18750 7300
+Wire Wire Line
+	18750 7300 18750 6800
 Connection ~ 15000 1750
 Wire Wire Line
@@
 Connection ~ 17500 3750
 Wire Wire Line
-	19800 6500 20000 6500
-Wire Wire Line
-	20000 6500 20000 7000
-Wire Wire Line
-	20000 7000 19700 7000
+	19800 6800 20000 6800
+Wire Wire Line
+	20000 6800 20000 7300
+Wire Wire Line
+	20000 7300 19700 7300
 Wire Wire Line
 	11750 6500 16000 6500
@@
 Text Label 18500 5200 2    98   ~ 0
 REF-3V3
-Text Label 21000 5000 2    98   ~ 0
+Text Label 21250 5000 2    98   ~ 0
 max4V1
 Wire Wire Line
-	21000 5000 20150 5000
+	21250 5000 20500 5000
 $Comp
 L eo-engine:#метка-3V3 #3V2
 U 1 1 642842BE
-P 18500 5400
-F 0 "#3V2" H 18500 5350 50  0001 C CNN
-F 1 "#метка-3V3" H 18450 5250 50  0001 C CNN
-F 2 "" H 18500 5400 50  0001 C CNN
-F 3 "" H 18500 5400 50  0001 C CNN
-	1    18500 5400
+P 18250 5500
+F 0 "#3V2" H 18250 5450 50  0001 C CNN
+F 1 "#метка-3V3" H 18200 5350 50  0001 C CNN
+F 2 "" H 18250 5500 50  0001 C CNN
+F 3 "" H 18250 5500 50  0001 C CNN
+	1    18250 5500
 	0    -1   -1   0
 $EndComp
-Wire Wire Line
-	18500 5400 19000 5400
 Wire Wire Line
 	17500 4500 17500 5000
@@
 Text Label 18900 5000 2    98   ~ 0
 LDO-DIRECT
-Wire Wire Line
-	18500 5600 18500 6200
 $Comp
 L eo-engine:Резистор*10кОм*0603 R33
 U 1 1 6436F649
-P 20800 6500
-F 0 "R33" H 21100 6300 138 0000 C CNN
-F 1 "Резистор*1кОм*0603" H 20800 7100 50  0001 C CNN
-F 2 "N_RLC:Резистор_SMD_0603_0,065_Вт_pnp" H 20900 7000 50  0001 C CNN
-F 3 "" V 20800 6500 50  0001 C CNN
-F 4 "1к" H 21100 6750 138 0000 C CNN "INFO"
-	1    20800 6500
+P 20800 6800
+F 0 "R33" H 21100 6600 138 0000 C CNN
+F 1 "Резистор*1кОм*0603" H 20800 7400 50  0001 C CNN
+F 2 "N_RLC:Резистор_SMD_0603_0,065_Вт_pnp" H 20900 7300 50  0001 C CNN
+F 3 "" V 20800 6800 50  0001 C CNN
+F 4 "1к" H 21100 7050 138 0000 C CNN "INFO"
+	1    20800 6800
 	-1   0    0    1
 $EndComp
 Wire Wire Line
-	20200 6500 20000 6500
-Connection ~ 20000 6500
-Wire Wire Line
-	21550 7000 21550 7250
-Wire Wire Line
-	21550 6700 21550 6500
-Wire Wire Line
-	21550 6500 21750 6500
-Wire Wire Line
-	21750 6500 21750 7250
-Wire Wire Line
-	21750 7250 21550 7250
-Wire Wire Line
-	21250 6700 21250 6500
-Wire Wire Line
-	21250 6500 21000 6500
-Wire Wire Line
-	21250 7000 21250 7250
-Wire Wire Line
-	21250 7250 21000 7250
-Wire Wire Line
-	21000 7250 21000 6500
+	20200 6800 20000 6800
+Connection ~ 20000 6800
+Wire Wire Line
+	21550 7300 21550 7550
+Wire Wire Line
+	21550 7000 21550 6800
+Wire Wire Line
+	21550 6800 21750 6800
+Wire Wire Line
+	21750 6800 21750 7550
+Wire Wire Line
+	21750 7550 21550 7550
+Wire Wire Line
+	21250 7000 21250 6800
+Wire Wire Line
+	21250 6800 21000 6800
+Wire Wire Line
+	21250 7300 21250 7550
+Wire Wire Line
+	21250 7550 21000 7550
+Wire Wire Line
+	21000 7550 21000 6800
 $Comp
 L eo-engine:Конденсатор*0,1мкФ*25В*0603 C15
 U 1 1 6447DC05
-P 22000 5250
-F 0 "C15" H 22184 5134 138 0000 L CNN
-F 1 "Конденсатор*0,1мкФ*25В*0603" H 21900 5550 50  0001 C CNN
-F 2 "N_RLC:Конденсатор_SMD_IEC_0603" H 22000 5450 50  0001 C CNN
-F 3 "" H 22000 5250 50  0001 C CNN
-F 4 "0,1мкФ 25В" H 22100 4800 138 0000 L CNN "INFO"
-F 5 "https://www.terraelectronica.ru/product/863311" H 22000 5450 50  0001 C CNN "LINK"
-F 6 "0,22" H 22000 5250 50  0001 C CNN "COST"
-	1    22000 5250
-	1    0    0    -1
-$EndComp
-Text Label 18500 5600 0    138  ~ 0
+P 20500 5250
+F 0 "C15" H 20684 5134 138 0000 L CNN
+F 1 "Конденсатор*0,1мкФ*25В*0603" H 20400 5550 50  0001 C CNN
+F 2 "N_RLC:Конденсатор_SMD_IEC_0603" H 20500 5450 50  0001 C CNN
+F 3 "" H 20500 5250 50  0001 C CNN
+F 4 "0,1мкФ 25В" H 20600 4800 138 0000 L CNN "INFO"
+F 5 "https://www.terraelectronica.ru/product/863311" H 20500 5450 50  0001 C CNN "LINK"
+F 6 "0,22" H 20500 5250 50  0001 C CNN "COST"
+	1    20500 5250
+	1    0    0    -1
+$EndComp
+Text Label 20000 6000 2    138  ~ 0
 COM
-Text Label 22000 6000 0    138  ~ 0
-COM
-Text Label 22000 5000 2    98   ~ 0
-max4V1
-Wire Wire Line
-	22000 5000 22000 5250
-Wire Wire Line
-	22000 5750 22000 6000
+Wire Wire Line
+	20500 5000 20500 5250
+Wire Wire Line
+	20500 5750 20500 6000
 $Comp
 L eo-engine:Конденсатор*0,1мкФ*25В*0603 C16
@@
 $EndComp
 Wire Wire Line
-	21000 6500 20800 6500
-Connection ~ 21000 6500
-Text Label 22500 6500 2    98   ~ 0
+	21000 6800 20800 6800
+Connection ~ 21000 6800
+Text Label 22500 6800 2    98   ~ 0
 max4V1
 Wire Wire Line
-	22500 6500 21750 6500
+	22500 6800 21750 6800
+Connection ~ 21750 6800
+Text Notes 24000 7000 0    138  ~ 0
+питание 2,5В для i2c датчиков
+$Comp
+L eo-engine:Микросхема*LDO*IN8V*OUT3V3*1,2A*SOT-223 G2
+U 1 1 6406D2CB
+P 8900 8950
+F 0 "G2" H 9900 9300 138 0000 C CNN
+F 1 "Микросхема*LDO*IN8V*OUT2V5*1,2A*SOT-223" H 9500 7900 50  0001 C CNN
+F 2 "N_VD_HL:Транзистор_NPN_SOT223_pnp" H 8900 9150 50  0001 C CNN
+F 3 "https://static.chipdip.ru/lib/432/DOC004432359.pdf" H 8900 9150 50  0001 C CNN
+F 4 "https://www.chipdip.ru/product/ld1117s25ctr" H 8900 8950 50  0001 C CNN "LINK"
+F 5 "LDO 2V5" H 9900 8300 138 0000 C CNN "INFO"
+	1    8900 8950
+	1    0    0    -1
+$EndComp
+Wire Wire Line
+	16000 6500 16000 5200
+Wire Wire Line
+	16000 5200 16500 5200
+Connection ~ 16500 5200
+Wire Wire Line
+	18250 5500 18250 5400
+Wire Wire Line
+	18250 5400 19000 5400
+Wire Wire Line
+	18500 5600 18500 6000
+NoConn ~ 20150 5200
+NoConn ~ 20150 5400
+NoConn ~ 20150 5600
+Connection ~ 20500 5000
+Wire Wire Line
+	20500 5000 20150 5000
+Connection ~ 18500 6000
+Wire Wire Line
+	18500 6000 18500 6500
+Wire Wire Line
+	18500 6000 20500 6000
 Wire Bus Line
 	3000 2850 3000 6400
-Connection ~ 21750 6500
-Text Notes 24000 7000 0    138  ~ 0
-питание 2,5В для i2c датчиков
 $EndSCHEMATC
