File: mag/mag.sch (KiCad schematic (older format))
At the start: 78 parts, among them K1 Кнопка_KLS7-TS5401-1.35-250-T, K2 Кнопка_KLS7-TS5401-1.35-250-T, X1 отверстие_под_пайку, X2 отверстие_под_пайку, X3 отверстие_под_пайку, X4 отверстие_под_пайку

Commit message: схема включения 2.5В по кнопке
Parts:
- added C1: Конденсатор*0,1мкФ*25В*0603, N_RLC:Конденсатор_SMD_IEC_0603, symbol eo-engine:Конденсатор*0,1мкФ*25В*0603
- added C2: Конденсатор*10мкФ*16В*0805, N_RLC:Конденсатор_SMD_IEC_0805, symbol eo-engine:Конденсатор*10мкФ*16В*0805
- added R1, R3: Резистор*1кОм*0603, N_RLC:Резистор_SMD_0603_0,065_Вт_pnp, symbol eo-engine:Резистор*10кОм*0603
- added R2: Резистор*10кОм*0603, N_RLC:Резистор_SMD_0603_0,065_Вт_pnp, symbol eo-engine:Резистор*10кОм*0603
- added VT1: Транзистор*pnp*0,5А*45В*SOT23, N_VD_HL:Корпус_КТ-46, symbol eo-engine:Транзистор*pnp*0,5А*45В*SOT23
- added VT11: Транзистор_полевой_N-канальный_КП526А9, MOTOR_VD_VT_HL:Корпус_КТ-46, symbol elements_2020:Транзистор_полевой_N-канальный_КП526А9
Connections:
- net GND: now also G2.1 (GND), C1.2, C2.2, R2.1, VT11.2
- net max4V1: now also VT1.2
- net TURN: now reaches K1.1, K1.2, R33.1
- net TURN: now also R3.1
- net 2V5: now reaches G2.2 (OUT(2V5))
- net 2V5: now also G2.4 (OUT(2V5)), C2.1
- net at G2.3 (IN): now also C1.1, VT1.3
- new net: R1.1, VT1.1
- new net: R1.2, VT11.3
- new net: R2.2, R3.2, VT11.1
Other:
- moved on the sheet: C14, G2

Commit message: инициирована замена транзисторов pnp на p-канальные
Parts:
- removed C1: Конденсатор*0,1мкФ*25В*0603, N_RLC:Конденсатор_SMD_IEC_0603, symbol eo-engine:Конденсатор*0,1мкФ*25В*0603
- removed C2: Конденсатор*10мкФ*16В*0805, N_RLC:Конденсатор_SMD_IEC_0805, symbol eo-engine:Конденсатор*10мкФ*16В*0805
- removed G2: Микросхема*LDO*IN8V*OUT2V5*1,2A*SOT-223, N_VD_HL:Транзистор_NPN_SOT223_pnp, symbol eo-engine:Микросхема*LDO*IN8V*OUT3V3*1,2A*SOT-223
- removed R1, R3: Резистор*1кОм*0603, N_RLC:Резистор_SMD_0603_0,065_Вт_pnp, symbol eo-engine:Резистор*10кОм*0603
- removed R2: Резистор*10кОм*0603, N_RLC:Резистор_SMD_0603_0,065_Вт_pnp, symbol eo-engine:Резистор*10кОм*0603
- removed VD3, VD5: Стабилитрон*3,3В*SOD80, N_VD_HL:SOD-80, symbol eo-engine:Стабилитрон*3,3В*SOD80
- removed VT1, VT2, VT6: Транзистор*pnp*0,5А*45В*SOT23, N_VD_HL:Корпус_КТ-46, symbol eo-engine:Транзистор*pnp*0,5А*45В*SOT23
- removed VT11: Транзистор_полевой_N-канальный_КП526А9, MOTOR_VD_VT_HL:Корпус_КТ-46, symbol elements_2020:Транзистор_полевой_N-канальный_КП526А9
- added R34, R8: Резистор*1кОм*0603, N_RLC:Резистор_SMD_0603_0,065_Вт_pnp, symbol eo-engine:Резистор*10кОм*0603
- added VD8: Стабилитрон*2,4В*SOD80, N_VD_HL:SOD-80, symbol eo-engine:Стабилитрон*3,3В*SOD80
- added VT12, VT2, VT6: Транзистор_полевой_P-канал(IRLML2246TRPBF), N_VD_HL:Корпус_КТ-46, symbol elements:Транзистор_полевой_P-канал(IRLML2246TRPBF)
- added VT13: Транзистор_полевой_N-канальный_КП526А9, MOTOR_VD_VT_HL:Корпус_КТ-46, symbol elements_2020:Транзистор_полевой_N-канальный_КП526А9
- R16, R33: value Резистор*1кОм*0603 -> Резистор*10кОм*0603; INFO 1к -> 10к
- R19: value Резистор*2,4кОм*0603 -> Резистор*7,5кОм*0603; INFO 2,4к -> 7,5к
- R20: value Резистор*10кОм*0603 -> Резистор*11кОм*0603; INFO 10к -> 11к
- VD2, VD7: value Стабилитрон*3,3В*SOD80 -> Стабилитрон*2,4В*SOD80; COST 1,7 -> 3; INFO 3,3В -> 2,4В; LINK https://www.terraelectronica.ru/product/311780 -> https://www.chipdip.ru/product/bzv55c2v4
Connections:
- net 5V: now also R10.1, VT12.2
- net CUR-DIRECT: now also VT12.1
- net GND: now also DA3.4 (GND), R33.1, VD8.1, VT13.2
- net REF-3V3: no longer C4.1, DA1.6, R4.2, R5.1, VD2.2
- net VOL-DIRECT: now also VT2.1
- net BUTT-TURN: now reaches R30.2, VT8.1
- net BUTT-TURN: now also K1.1, K1.2; no longer R33.2
- net max0.22A: now reaches R16.1
- net max0.22A: now also VT12.3, VT2.2
- removed net COM: C15.2, DA3.4 (GND), VT8.3
- net REF-0V1 renamed REF-0V22
- removed net TURN: K1.1, K1.2, R33.1
- net max4V1 renamed max4V
- net max4V: now also R8.1, VT2.3, VT6.2; no longer C15.1, DA3.8 (VCC), VT10.2, VT9.2
- new net: VT10.2, VT9.2
- new net BAT-REF-2V4: R34.2, VD8.2
- new net DIRECT: R8.2, VT13.3, VT6.1, VT8.3
- new net ESP-TURN: R33.2, VT13.1
- new net REF-2V4: C4.1, DA1.6, R4.2, R5.1, VD2.2
- new net VBAT: C15.1, DA3.8 (VCC), R34.1, VT6.3
Other:
- moved on the sheet: C15, C16, DA3, K1, R10, R16, R30, R31, R32, VD7, VT10, VT8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
